Commit message: renamed xacro files for better readability

File: urdf/robotiq_hande_gripper.xacro (robot description, xacro)
@@ -1,7 +1,134 @@
 <?xml version="1.0"?>
-<robot xmlns:xacro="http://ros.org/wiki/xacro"
-       name="robotiq_hande_gripper" >
-  <xacro:include filename="$(find robotiq_hande_description)/urdf/robotiq_hande_gripper.urdf.xacro" />
-  <link name="tool0" />
-  <xacro:robotiq_hande_gripper parent="tool0" prefix="" />
+<robot xmlns:xacro="http://ros.org/wiki/xacro">
+  <!--
+    Based on the URDF file by Cristian C Beltran-Hernandez
+  -->
+  <xacro:include filename="$(find robotiq_hande_description)/urdf/materials.xacro" />
+  <xacro:macro name="robotiq_hande_gripper" params="prefix parent">
+    <!-- Robotiq Coupler -->
+    <!--  + Height added by the coupler: 13.9mm -->
+    <!--  + Reference frame: at the middle (6.95mm) -->
+    <joint name="robotiq_coupler_joint" type="fixed">
+      <origin xyz="0 0 0.00695" rpy="0 0 ${-pi/2.0}" />
+      <parent link="${parent}"/>
+      <child link="robotiq_coupler"/>
+    </joint>
+    <link name="${prefix}robotiq_coupler">
+      <inertial>
+        <mass value="0.168" />
+        <inertia
+          ixx="6.17674E-05" ixy="0.0" ixz="0.0"
+          iyy="6.17674E-05" iyz="0.0"
+          izz="1.18125E-04"
+        />
+      </inertial>
+      <collision>
+        <geometry>
+          <cylinder length="0.0139" radius="0.0375"/>
+        </geometry>
+      </collision>
+      <visual>
+        <geometry>
+          <mesh filename="package://robotiq_hande_description/meshes/coupler.dae" />
+        </geometry>
+        <material name="DarkGrey" />
+      </visual>
+    </link>
+    <joint name="${prefix}robotiq_hande_base_joint" type="fixed">
+      <origin rpy="0 0 0" xyz="0 0 0.055"/>
+      <parent link="${prefix}robotiq_coupler"/>
+      <child link="${prefix}hande_link"/>
+    </joint>
+    <link name="${prefix}hande_link">
+      <inertial>
+        <mass value="0.86387"/>
+        <inertia
+          ixx="0.001" ixy="0.0" ixz="0.0"
+          iyy="0.001" iyz="0.0"
+          izz="0.0006"
+        />
+      </inertial>
+      <collision>
+        <geometry>
+          <cylinder length="0.0988" radius="0.0375"/>
+        </geometry>
+      </collision>
+      <visual>
+        <origin rpy="0 -1.570796 -1.570796" xyz="0 0 -0.0016"/>
+        <geometry>
+          <mesh filename="package://robotiq_hande_description/meshes/hande.dae" scale="1.0 1.0 1.0"/>
+        </geometry>
+        <material name="DarkGrey"/>
+      </visual>
+    </link>
+    <joint name="${prefix}hande_left_finger_joint" type="prismatic">
+      <origin rpy="0 0 0" xyz="0 0 0.0345"/>
+      <parent link="${prefix}hande_link"/>
+      <child link="${prefix}hande_left_finger"/>
+      <axis xyz="0 1 0"/>
+      <limit effort="130" lower="-0.025" upper="0" velocity="0.15"/>
+    </joint>
+    <link name="${prefix}hande_left_finger">
+      <inertial>
+        <origin rpy="0 0 0" xyz="0 0 0"/>
+        <mass value="0.03804"/>
+        <inertia
+          ixx="1E-9" ixy="0.0" ixz="0.0"
+          iyy="1E-9" iyz="0.0"
+          izz="1E-9"
+        />
+      </inertial>
+      <collision>
+        <origin rpy="0 0 3.1415926" xyz="0 0 0"/>
+        <geometry>
+          <mesh filename="package://robotiq_hande_description/meshes/finger_collision.dae" scale="1.0 1.0 1.0"/>
+        </geometry>
+      </collision>
+      <visual>
+        <origin rpy="1.570796 0 3.1415926" xyz="0 0 0"/>
+        <geometry>
+          <mesh filename="package://robotiq_hande_description/meshes/finger.dae" scale="1.0 1.0 1.0"/>
+        </geometry>
+        <material name="Grey"/>
+      </visual>
+    </link>
+    <joint name="${prefix}hande_right_finger_joint" type="prismatic">
+      <origin rpy="0 0 0" xyz="0 0 0.0345"/>
+      <parent link="${prefix}hande_link"/>
+      <child link="${prefix}hande_right_finger"/>
+      <axis xyz="0 -1 0"/>
+      <limit effort="130" lower="-0.025" upper="0" velocity="0.15"/>
+      <mimic joint="${prefix}hande_left_finger_joint" multiplier="1" offset="0"/>
+    </joint>
+    <link name="${prefix}hande_right_finger">
+      <inertial>
+        <origin rpy="0 0 0" xyz="0 0 0"/>
+        <mass value="0.03804"/>
+        <inertia
+          ixx="1E-9" ixy="0.0" ixz="0.0"
+          iyy="1E-9" iyz="0.0"
+          izz="1E-9"
+        />
+      </inertial>
+      <collision>
+        <origin rpy="0 0 0" xyz="0 0 0"/>
+        <geometry>
+          <mesh filename="package://robotiq_hande_description/meshes/finger_collision.dae" scale="1.0 1.0 1.0"/>
+        </geometry>
+      </collision>
+      <visual>
+        <origin rpy="1.570796 0 0" xyz="0 0 0"/>
+        <geometry>
+          <mesh filename="package://robotiq_hande_description/meshes/finger.dae" scale="1.0 1.0 1.0"/>
+        </geometry>
+        <material name="Grey" />
+      </visual>
+    </link>
+    <joint name="${prefix}robotiq_hande_end_joint" type="fixed">
+      <origin rpy="0 0 0" xyz="0 0 0.095"/>
+      <parent link="${prefix}hande_link"/>
+      <child link="${prefix}hande_end"/>
+    </joint>
+    <link name="${prefix}hande_end" />
+  </xacro:macro>
 </robot>

Commit message: typo for prefix arg

File: urdf/robotiq_hande_gripper.xacro (robot description, xacro)
@@ -12,5 +12,5 @@
       <origin xyz="0 0 0.00695" rpy="0 0 ${-pi/2.0}" />
       <parent link="${parent}"/>
-      <child link="robotiq_coupler"/>
+      <child link="${prefix}robotiq_coupler"/>
     </joint>
     <link name="${prefix}robotiq_coupler">

Commit message: changed grip width offset by +25mm

File: urdf/robotiq_hande_gripper.xacro (robot description, xacro)
@@ -63,9 +63,9 @@
     </link>
     <joint name="${prefix}hande_left_finger_joint" type="prismatic">
-      <origin rpy="0 0 0" xyz="0 0 0.0345"/>
+      <origin rpy="0 0 0" xyz="0 -0.025 0.0345"/>
       <parent link="${prefix}hande_link"/>
       <child link="${prefix}hande_left_finger"/>
       <axis xyz="0 1 0"/>
-      <limit effort="130" lower="-0.025" upper="0" velocity="0.15"/>
+      <limit effort="130" lower="0" upper="0.025" velocity="0.15"/>
     </joint>
     <link name="${prefix}hande_left_finger">
@@ -94,9 +94,9 @@
     </link>
     <joint name="${prefix}hande_right_finger_joint" type="prismatic">
-      <origin rpy="0 0 0" xyz="0 0 0.0345"/>
+      <origin rpy="0 0 0" xyz="0 0.025 0.0345"/>
       <parent link="${prefix}hande_link"/>
       <child link="${prefix}hande_right_finger"/>
       <axis xyz="0 -1 0"/>
-      <limit effort="130" lower="-0.025" upper="0" velocity="0.15"/>
+      <limit effort="130" lower="0" upper="0.025" velocity="0.15"/>
       <mimic joint="${prefix}hande_left_finger_joint" multiplier="1" offset="0"/>
     </joint>
