Commit message: added param frequency_hz

File: urdf/robotiq_hande_gripper.ros2_control.xacro (robot description, xacro)
@@ -1,5 +1,5 @@
 <?xml version="1.0"?>
 <robot xmlns:xacro="http://www.ros.org/wiki/xacro">
-  <xacro:macro name="robotiq_hande_ros2_control" params="name prefix grip_pos_min grip_pos_max tty baudrate parity data_bits stop_bit slave_id use_fake_hardware">
+  <xacro:macro name="robotiq_hande_ros2_control" params="name prefix grip_pos_min grip_pos_max tty baudrate parity data_bits stop_bit slave_id frequency_hz use_fake_hardware">
     <ros2_control name="${name}" type="system">
       <hardware>
@@ -17,4 +17,5 @@
           <param name="stop_bit">${stop_bit}</param>
           <param name="slave_id">${slave_id}</param>
+          <param name="frequency_hz">${frequency_hz}</param>
         </xacro:unless>
       </hardware>

File: urdf/robotiq_hande_gripper.urdf.xacro (robot description, xacro)
@@ -10,4 +10,5 @@
   <xacro:arg name="stop_bit" default="1"/>
   <xacro:arg name="slave_id" default="9"/>
+  <xacro:arg name="frequency_hz" default="10"/>
   <xacro:arg name="use_fake_hardware" default="true"/>
   <xacro:include filename="$(find robotiq_hande_description)/urdf/robotiq_hande_gripper.xacro"/>
@@ -25,4 +26,5 @@
     stop_bit="$(arg stop_bit)"
     slave_id="$(arg slave_id)"
+    frequency_hz="$(arg frequency_hz)"
     use_fake_hardware="$(arg use_fake_hardware)"
   />

File: urdf/robotiq_hande_gripper.xacro (robot description, xacro)
@@ -20,4 +20,5 @@
             slave_id
             use_fake_hardware
+            frequency_hz:=10
             coupler_mass:=0.119
             xyz:='0 0 0'
@@ -36,4 +37,5 @@
       stop_bit="${stop_bit}"
       slave_id="${slave_id}"
+      frequency_hz="${frequency_hz}"
       use_fake_hardware="${use_fake_hardware}"
     />

Commit message: hande: changed `tty` to `tty_port`

File: urdf/robotiq_hande_gripper.ros2_control.xacro (robot description, xacro)
@@ -1,5 +1,5 @@
 <?xml version="1.0"?>
 <robot xmlns:xacro="http://www.ros.org/wiki/xacro">
-  <xacro:macro name="robotiq_hande_ros2_control" params="name prefix grip_pos_min grip_pos_max tty baudrate parity data_bits stop_bit slave_id frequency_hz use_fake_hardware">
+  <xacro:macro name="robotiq_hande_ros2_control" params="name prefix grip_pos_min grip_pos_max tty_port baudrate parity data_bits stop_bit slave_id frequency_hz use_fake_hardware">
     <ros2_control name="${name}" type="system">
       <hardware>
@@ -11,5 +11,5 @@
           <param name="grip_pos_min">${grip_pos_min}</param>
           <param name="grip_pos_max">${grip_pos_max}</param>
-          <param name="tty">${tty}</param>
+          <param name="tty_port">${tty_port}</param>
           <param name="baudrate">${baudrate}</param>
           <param name="parity">${parity}</param>

File: urdf/robotiq_hande_gripper.urdf.xacro (robot description, xacro)
@@ -4,5 +4,5 @@
   <xacro:arg name="grip_pos_min" default="0"/>
   <xacro:arg name="grip_pos_max" default="0.025"/>
-  <xacro:arg name="tty" default="/tmp/ttyUR"/>
+  <xacro:arg name="tty_port" default="/tmp/ttyUR"/>
   <xacro:arg name="baudrate" default="115200"/>
   <xacro:arg name="parity" default="N"/>
@@ -20,5 +20,5 @@
     grip_pos_min="$(arg grip_pos_min)"
     grip_pos_max="$(arg grip_pos_max)"
-    tty="$(arg tty)"
+    tty_port="$(arg tty_port)"
     baudrate="$(arg baudrate)"
     parity="$(arg parity)"

File: urdf/robotiq_hande_gripper.xacro (robot description, xacro)
@@ -13,5 +13,5 @@
             grip_pos_min
             grip_pos_max
-            tty
+            tty_port
             baudrate
             parity
@@ -31,5 +31,5 @@
       grip_pos_min="${grip_pos_min}"
       grip_pos_max="${grip_pos_max}"
-      tty="${tty}"
+      tty_port="${tty_port}"
       baudrate="${baudrate}"
       parity="${parity}"

Commit message: renamed virtual_tty to socat_tty

File: urdf/robotiq_hande_gripper.ros2_control.xacro (robot description, xacro)
@@ -1,5 +1,5 @@
 <?xml version="1.0"?>
 <robot xmlns:xacro="http://www.ros.org/wiki/xacro">
-  <xacro:macro name="robotiq_hande_ros2_control" params="name prefix grip_pos_min grip_pos_max tty_port baudrate parity data_bits stop_bit slave_id frequency_hz use_fake_hardware">
+  <xacro:macro name="robotiq_hande_ros2_control" params="name prefix grip_pos_min grip_pos_max tty_port baudrate parity data_bits stop_bit slave_id frequency_hz create_socat_tty ip_adress port use_fake_hardware">
     <ros2_control name="${name}" type="system">
       <hardware>
@@ -18,7 +18,7 @@
           <param name="slave_id">${slave_id}</param>
           <param name="frequency_hz">${frequency_hz}</param>
-          <param name="virtual_tty">true</param>
-          <param name="ip_adress">aegis_ur</param>
-          <param name="port">54321</param>
+          <param name="create_socat_tty">${create_socat_tty}</param>
+          <param name="ip_adress">${ip_adress}</param>
+          <param name="port">${port}</param>
         </xacro:unless>
       </hardware>

File: urdf/robotiq_hande_gripper.urdf.xacro (robot description, xacro)
@@ -11,4 +11,7 @@
   <xacro:arg name="slave_id" default="9"/>
   <xacro:arg name="frequency_hz" default="10"/>
+  <xacro:arg name="create_socat_tty" default="false"/>
+  <xacro:arg name="ip_adress" default="192.168.100.10"/>
+  <xacro:arg name="port" default="54321"/>
   <xacro:arg name="use_fake_hardware" default="true"/>
   <xacro:include filename="$(find robotiq_hande_description)/urdf/robotiq_hande_gripper.xacro"/>
@@ -27,4 +30,7 @@
     slave_id="$(arg slave_id)"
     frequency_hz="$(arg frequency_hz)"
+    create_socat_tty="$(arg create_socat_tty)"
+    ip_adress="$(arg ip_adress)"
+    port="$(arg port)"
     use_fake_hardware="$(arg use_fake_hardware)"
   />

File: urdf/robotiq_hande_gripper.xacro (robot description, xacro)
@@ -21,4 +21,7 @@
             use_fake_hardware
             frequency_hz:=10
+            create_socat_tty:=false
+            ip_adress:=192.168.100.10
+            port:=54321
             coupler_mass:=0.119
             xyz:='0 0 0'
@@ -38,4 +41,7 @@
       slave_id="${slave_id}"
       frequency_hz="${frequency_hz}"
+      create_socat_tty="${create_socat_tty}"
+      ip_adress="${ip_adress}"
+      port="${port}"
       use_fake_hardware="${use_fake_hardware}"
     />

Commit message: fmt

File: urdf/robotiq_hande_gripper.ros2_control.xacro (robot description, xacro)
@@ -1,5 +1,8 @@
 <?xml version="1.0"?>
 <robot xmlns:xacro="http://www.ros.org/wiki/xacro">
-  <xacro:macro name="robotiq_hande_ros2_control" params="name prefix grip_pos_min grip_pos_max tty_port baudrate parity data_bits stop_bit slave_id frequency_hz create_socat_tty ip_adress port use_fake_hardware">
+  <xacro:macro
+    name="robotiq_hande_ros2_control"
+    params="name prefix grip_pos_min grip_pos_max tty_port baudrate parity data_bits stop_bit slave_id frequency_hz create_socat_tty ip_adress port use_fake_hardware"
+  >
     <ros2_control name="${name}" type="system">
       <hardware>

Commit message: Humble release (#16)
* Update CHANGELOG.md

* FIX: change inertial macro name to avoid namespace collisions (#6)

* FIX: change inertial macro name to avoid namespace collisions

* CHG: docs

* CHG: pre-commit

* Update urdf/robotiq_hande_gripper.xacro

Co-authored-by: Maciej Aleksandrowicz <mac.aleksandrowicz@gmail.com>

* REV: cylinder_inertial filename

---------

Co-authored-by: Maciej Aleksandrowicz <mac.aleksandrowicz@gmail.com>

* CHG: changelog

* CHG: package version bump

* added citation file

* bumped version

* fixed default rotatation of hande

* updated citation file

* CHG: changelog

* Make gripper mounting pose configurable

* Format

* Format

* Format

* Update changelog

* Update changelog

Co-authored-by: Maciej Aleksandrowicz <mac.aleksandrowicz@gmail.com>

* added param frequency_hz

* hande: changed `tty` to `tty_port`

* added socat params

* renamed virtual_tty to socat_tty

* updated cmake version

* fmt

* updated changelog

* updated changelog

* Merge pull request #15 from AGH-CEAI/bugfix/fix_typo

Fix typo

* CHG: bump version

* FIX: docs

* CHG: bumb citation version

---------

Co-authored-by: Maciej Aleksandrowicz <mac.aleksandrowicz@gmail.com>
Co-authored-by: Jakub <sivral@proton.me>

File: urdf/robotiq_hande_gripper.ros2_control.xacro (robot description, xacro)
@@ -1,5 +1,8 @@
 <?xml version="1.0"?>
 <robot xmlns:xacro="http://www.ros.org/wiki/xacro">
-  <xacro:macro name="robotiq_hande_ros2_control" params="name prefix grip_pos_min grip_pos_max tty baudrate parity data_bits stop_bit slave_id use_fake_hardware">
+  <xacro:macro
+    name="robotiq_hande_ros2_control"
+    params="name prefix grip_pos_min grip_pos_max tty_port baudrate parity data_bits stop_bit slave_id frequency_hz create_socat_tty socat_ip_address socat_port use_fake_hardware"
+  >
     <ros2_control name="${name}" type="system">
       <hardware>
@@ -11,5 +14,5 @@
           <param name="grip_pos_min">${grip_pos_min}</param>
           <param name="grip_pos_max">${grip_pos_max}</param>
-          <param name="tty">${tty}</param>
+          <param name="tty_port">${tty_port}</param>
           <param name="baudrate">${baudrate}</param>
           <param name="parity">${parity}</param>
@@ -17,4 +20,8 @@
           <param name="stop_bit">${stop_bit}</param>
           <param name="slave_id">${slave_id}</param>
+          <param name="frequency_hz">${frequency_hz}</param>
+          <param name="create_socat_tty">${create_socat_tty}</param>
+          <param name="socat_ip_address">${socat_ip_address}</param>
+          <param name="socat_port">${socat_port}</param>
         </xacro:unless>
       </hardware>

File: urdf/robotiq_hande_gripper.urdf.xacro (robot description, xacro)
@@ -4,5 +4,5 @@
   <xacro:arg name="grip_pos_min" default="0"/>
   <xacro:arg name="grip_pos_max" default="0.025"/>
-  <xacro:arg name="tty" default="/tmp/ttyUR"/>
+  <xacro:arg name="tty_port" default="/tmp/ttyUR"/>
   <xacro:arg name="baudrate" default="115200"/>
   <xacro:arg name="parity" default="N"/>
@@ -10,4 +10,8 @@
   <xacro:arg name="stop_bit" default="1"/>
   <xacro:arg name="slave_id" default="9"/>
+  <xacro:arg name="frequency_hz" default="10"/>
+  <xacro:arg name="create_socat_tty" default="false"/>
+  <xacro:arg name="socat_ip_address" default="192.168.100.10"/>
+  <xacro:arg name="socat_port" default="54321"/>
   <xacro:arg name="use_fake_hardware" default="true"/>
   <xacro:include filename="$(find robotiq_hande_description)/urdf/robotiq_hande_gripper.xacro"/>
@@ -19,5 +23,5 @@
     grip_pos_min="$(arg grip_pos_min)"
     grip_pos_max="$(arg grip_pos_max)"
-    tty="$(arg tty)"
+    tty_port="$(arg tty_port)"
     baudrate="$(arg baudrate)"
     parity="$(arg parity)"
@@ -25,4 +29,8 @@
     stop_bit="$(arg stop_bit)"
     slave_id="$(arg slave_id)"
+    frequency_hz="$(arg frequency_hz)"
+    create_socat_tty="$(arg create_socat_tty)"
+    socat_ip_address="$(arg socat_ip_address)"
+    socat_port="$(arg socat_port)"
     use_fake_hardware="$(arg use_fake_hardware)"
   />

File: urdf/robotiq_hande_gripper.xacro (robot description, xacro)
@@ -6,5 +6,26 @@
   <xacro:include filename="$(find robotiq_hande_description)/urdf/robotiq_hande_gripper.ros2_control.xacro"/>
   <xacro:include filename="$(find robotiq_hande_description)/urdf/cylinder_inertial.xacro"/>
-  <xacro:macro name="robotiq_hande_gripper" params="name prefix parent grip_pos_min grip_pos_max tty baudrate parity data_bits stop_bit slave_id use_fake_hardware coupler_mass:=0.119">
+  <xacro:macro
+    name="robotiq_hande_gripper"
+    params="name
+            prefix
+            parent
+            grip_pos_min
+            grip_pos_max
+            tty_port
+            baudrate
+            parity
+            data_bits
+            stop_bit
+            slave_id
+            use_fake_hardware
+            frequency_hz:=10
+            create_socat_tty:=false
+            socat_ip_address:=192.168.100.10
+            socat_port:=54321
+            coupler_mass:=0.119
+            xyz:='0 0 0'
+            rpy:='0 0 0'"
+  >
     <!-- ros2_control parameters  -->
     <xacro:robotiq_hande_ros2_control
@@ -13,5 +34,5 @@
       grip_pos_min="${grip_pos_min}"
       grip_pos_max="${grip_pos_max}"
-      tty="${tty}"
+      tty_port="${tty_port}"
       baudrate="${baudrate}"
       parity="${parity}"
@@ -19,4 +40,8 @@
       stop_bit="${stop_bit}"
       slave_id="${slave_id}"
+      frequency_hz="${frequency_hz}"
+      create_socat_tty="${create_socat_tty}"
+      socat_ip_address="${socat_ip_address}"
+      socat_port="${socat_port}"
       use_fake_hardware="${use_fake_hardware}"
     />
@@ -32,5 +57,5 @@
     <xacro:arg name="hande_radius" default="0.0375"/>
     <joint name="${prefix}robotiq_hande_coupler_joint" type="fixed">
-      <origin xyz="0 0 0" rpy="0 0 0"/>
+      <origin xyz="${xyz}" rpy="${rpy}"/>
       <parent link="${parent}"/>
       <child link="${prefix}robotiq_hande_coupler"/>
